File: Hardware/ZX_Gesture_Sensor_SMD.brd (EAGLE design)
At the start: 57.2 x 22.9 mm, 49 parts, among them Q1 MMBT2222A, Q2 MOSFET-NCHANNEL2N7002PW, U1 PIC16F1823-14PINTSSOP, U2 MCP6021T-E/OT, U3 DMC2700UDM, U4 DMC2700UDM, U6 TSOP57238TT1

Commit message: Updated Board File
Parts:
- added LOGO2: SFE_LOGO_FLAME.1_INCH, SparkFun-Aesthetics:SFE_LOGO_FLAME_.1
- moved FID2 3.59 mm to (52.6, 4.76)
- moved FID4 2.84 mm to (51.5, 2.73)
- moved U$5 2.81 mm to (12.1, 8.47)
- moved JP3 1.00 mm to (31.8, 0.00)
- moved JP1 1.00 mm to (16.5, 0.00)
- moved U$6 0.46 mm to (30.0, 8.64)
Routing:
- net ICSPDAT/DACOUT: track 52.4 -> 57.2 mm
- net UART_RX: track 37.4 -> 38.5 mm
- net ICSPCLK/DATA_RDY: track 43.7 -> 44.6 mm
- net VCC: track 112.8 -> 113.6 mm
- net I2C_SDA: track 46.4 -> 47.1 mm, vias 3 -> 2
Other:
- outline, holes or cut-outs redrawn
