File: Hardware/ZX_Gesture_Sensor_SMD.brd (EAGLE design)
At the start: 62.4 x 16.5 mm, 50 parts, among them Q1 MMBT2222A, Q2 MOSFET-NCHANNEL2N7002PW, U1 PIC16F1823-14PINTSSOP, U2 MCP6021T-E/OT, U3 DMC2700UDM, U4 DMC2700UDM, U5 TSSP57038

Commit message: Updated BRD File
Routing:
- net GND: vias 24 -> 25
Other:
- board size 62.4 x 16.5 mm -> 61.8 x 16.5 mm
Changed lines of the file:
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@@
 <setting verticaltext="up"/>
 </settings>
-<grid distance="0.00625" unitdist="inch" unit="inch" style="dots" multiple="1" display="yes" altdistance="0.005" altunitdist="inch" altunit="inch"/>
+<grid distance="0.025" unitdist="inch" unit="inch" style="dots" multiple="1" display="yes" altdistance="0.005" altunitdist="inch" altunit="inch"/>
 <layers>
 <layer number="1" name="Top" color="4" fill="1" visible="yes" active="yes"/>
@@
 <layer number="18" name="Vias" color="2" fill="1" visible="yes" active="yes"/>
 <layer number="19" name="Unrouted" color="6" fill="1" visible="yes" active="yes"/>
-<layer number="20" name="Dimension" color="15" fill="1" visible="no" active="yes"/>
-<layer number="21" name="tPlace" color="16" fill="1" visible="no" active="yes"/>
-<layer number="22" name="bPlace" color="14" fill="1" visible="no" active="yes"/>
+<layer number="20" name="Dimension" color="15" fill="1" visible="yes" active="yes"/>
+<layer number="21" name="tPlace" color="16" fill="1" visible="yes" active="yes"/>
+<layer number="22" name="bPlace" color="14" fill="1" visible="yes" active="yes"/>
 <layer number="23" name="tOrigins" color="15" fill="1" visible="no" active="yes"/>
 <layer number="24" name="bOrigins" color="15" fill="1" visible="no" active="yes"/>
@@
 <text x="38.19525" y="4.09575" size="0.8128" layer="21" font="vector" ratio="15">VCC</text>
 <text x="40.3225" y="3.65125" size="0.8128" layer="22" font="vector" ratio="15" rot="MR0">VCC</text>
-<wire x1="5.55625" y1="1.27" x2="51.27625" y2="1.27" width="0.2032" layer="20"/>
+<wire x1="6.19125" y1="1.27" x2="51.27625" y2="1.27" width="0.2032" layer="20"/>
 <wire x1="51.27625" y1="1.27" x2="51.435" y2="1.27" width="0.2032" layer="20"/>
 <text x="50.4825" y="1.905" size="1.016" layer="16" ratio="20" rot="MR0">v05</text>
-<wire x1="50.95875" y1="17.78" x2="5.23875" y2="17.78" width="0.2032" layer="20"/>
+<wire x1="50.95875" y1="17.78" x2="5.87375" y2="17.78" width="0.2032" layer="20"/>
 <wire x1="25.7175" y1="17.78" x2="26.035" y2="18.0975" width="0.254" layer="47"/>
-<wire x1="5.55625" y1="1.27" x2="5.23875" y2="17.78" width="0.2032" layer="20" curve="-181.090425"/>
+<wire x1="6.19125" y1="1.27" x2="5.87375" y2="17.78" width="0.2032" layer="20" curve="-181.090425"/>
 <wire x1="50.95875" y1="17.78" x2="51.27625" y2="1.27" width="0.2032" layer="20" curve="-181.090425"/>
 <dimension x1="2.54" y1="9.525" x2="54.61" y2="9.525" x3="28.575" y3="23.1775" textsize="1.778" layer="47" unit="inch"/>
@@
 <wire x1="9.2075" y1="7.2" x2="11.43" y2="7.2" width="0.254" layer="16"/>
 <polygon width="0.254" layer="1">
-<vertex x="-2.69875" y="5.08"/>
+<vertex x="-2.06375" y="5.08"/>
 <vertex x="2.54" y="1.27"/>
 <vertex x="54.61" y="1.27"/>
@@
 <vertex x="54.61" y="17.78"/>
 <vertex x="2.54" y="17.78"/>
-<vertex x="-2.69875" y="13.97"/>
+<vertex x="-2.06375" y="13.97"/>
 </polygon>
 <polygon width="0.254" layer="16">
-<vertex x="-2.69875" y="5.23875"/>
-<vertex x="-2.69875" y="14.12875"/>
+<vertex x="-2.06375" y="5.23875"/>
+<vertex x="-2.06375" y="14.12875"/>
 <vertex x="2.54" y="17.78"/>
 <vertex x="54.61" y="17.78"/>
@@
 <wire x1="21.6925" y1="5.3975" x2="21.59" y2="5.5" width="0.254" layer="16"/>
 <wire x1="10.09" y1="10.16" x2="13.97" y2="10.16" width="0.2032" layer="16"/>
+<via x="35.56" y="14.605" extent="1-16" drill="0.381"/>
 </signal>
 <signal name="I2C_SDA">
@@
 <wire x1="43.4975" y1="5.3975" x2="43.33875" y2="5.55625" width="0.254" layer="1"/>
 </signal>
-<signal name="N$27">
-<via x="35.56" y="14.605" extent="1-16" drill="0.381"/>
-</signal>
 </signals>
