File: Hardware/ZX_Gesture_Sensor_SMD_v02.brd (EAGLE design)
At the start: 57.2 x 19.1 mm, 51 parts, among them Q1 MMBT2222A, Q2 MOSFET-NCHANNEL2N7002PW, U1 PIC16F1823-14PINTSSOP, U2 MCP6021T-E/OT, U3 DMC2700UDM, U4 DMC2700UDM, U6 TSOP57238TT1

Commit message: Updated BRD file
Parts:
- moved FID4 12.8 mm to (51.5, 16.7)
- moved FID1 12.8 mm to (4.45, 3.56)
- moved TP4 2.54 mm to (34.3, 5.08)
- moved TP5 2.54 mm to (34.3, 7.62)
Routing:
- net ICSPDAT/DACOUT: track 25.1 -> 23.0 mm
- net ICSPCLK/DATA_RDY: track 30.5 -> 30.2 mm, vias 3 -> 4
- net GND: vias 18 -> 19
Changed lines of the file:
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@@
 <setting verticaltext="up"/>
 </settings>
-<grid distance="0.005" unitdist="inch" unit="inch" style="dots" multiple="1" display="yes" altdistance="0.005" altunitdist="inch" altunit="inch"/>
+<grid distance="0.05" unitdist="inch" unit="inch" style="dots" multiple="1" display="yes" altdistance="0.005" altunitdist="inch" altunit="inch"/>
 <layers>
 <layer number="1" name="Top" color="4" fill="1" visible="yes" active="yes"/>
@@
 <text x="28.6639" y="8.2804" size="0.8128" layer="22" font="vector" ratio="15" rot="MR180" align="bottom-center">I2C Addr</text>
 <text x="22.6314" y="16.3195" size="1.778" layer="21" font="vector" ratio="15" align="bottom-center">ZX Gesture</text>
-<text x="53.1495" y="14.9225" size="1.2192" layer="1" font="vector" ratio="15" rot="R135" align="center">v02</text>
+<text x="53.6575" y="14.4145" size="1.2192" layer="1" font="vector" ratio="15" rot="R135" align="center">v02</text>
 <text x="47.6885" y="2.667" size="0.8128" layer="22" font="vector" ratio="15" rot="MR0" align="bottom-center">I2C Pullups</text>
 <text x="18.4785" y="2.3495" size="0.8128" layer="21" font="vector" ratio="15" align="bottom-center">GRN</text>
@@
 </element>
 <element name="SJ2" library="SparkFun-Passives" package="PAD-JUMPER-2-NO_YES_SILK" value="JUMPER-PAD-2-NOYES_SILK" x="28.8925" y="6.0325" rot="MR180"/>
-<element name="FID1" library="SparkFun-Aesthetics" package="MICRO-FIDUCIAL" value="FIDUCIALUFIDUCIAL" x="5.715" y="16.256" rot="MR0"/>
+<element name="FID1" library="SparkFun-Aesthetics" package="MICRO-FIDUCIAL" value="FIDUCIALUFIDUCIAL" x="4.445" y="3.556" rot="MR0"/>
 <element name="FID2" library="SparkFun-Aesthetics" package="MICRO-FIDUCIAL" value="FIDUCIALUFIDUCIAL" x="54.229" y="5.3975" rot="MR0"/>
 <element name="U$5" library="SparkFun-Aesthetics" package="SFE_LOGO_NAME_FLAME_.1" value="SFE_LOGO_NAME_FLAME.1_INCH" x="13.2842" y="6.9469"/>
@@
 <element name="TP2" library="SparkFun-Passives" package="PAD.03X.04" value="TEST-POINT3X4" x="34.29" y="10.16" rot="MR0"/>
 <element name="TP3" library="SparkFun-Passives" package="PAD.03X.04" value="TEST-POINT3X4" x="34.29" y="15.24" rot="MR0"/>
-<element name="TP4" library="SparkFun-Passives" package="PAD.03X.04" value="TEST-POINT3X4" x="34.29" y="7.62" rot="MR0"/>
-<element name="TP5" library="SparkFun-Passives" package="PAD.03X.04" value="TEST-POINT3X4" x="34.29" y="5.08" rot="MR0"/>
+<element name="TP4" library="SparkFun-Passives" package="PAD.03X.04" value="TEST-POINT3X4" x="34.29" y="5.08" rot="MR0"/>
+<element name="TP5" library="SparkFun-Passives" package="PAD.03X.04" value="TEST-POINT3X4" x="34.29" y="7.62" rot="MR0"/>
 <element name="U$6" library="SparkFun-Aesthetics" package="GESTURESENSE_TEXT" value="GESTURESENSE_LOGOSTEXT" x="32.131" y="6.223"/>
 <element name="D1" library="SparkFun-LED" package="SFH4641-SHORT2" value="SFH4641SHORT2" x="9.525" y="9.525" rot="R270">
@@
 <attribute name="PROD_ID" value="RES-07856" x="47.9425" y="13.97" size="1.778" layer="28" font="vector" ratio="15" rot="MR0" display="off"/>
 </element>
-<element name="FID4" library="SparkFun-Aesthetics" package="MICRO-FIDUCIAL" value="FIDUCIALUFIDUCIAL" x="52.7685" y="4.0005"/>
+<element name="FID4" library="SparkFun-Aesthetics" package="MICRO-FIDUCIAL" value="FIDUCIALUFIDUCIAL" x="51.4985" y="16.7005"/>
 <element name="R13" library="SparkFun-Resistors" package="0603-RES" value="1K" x="9.8425" y="10.16" rot="MR180">
 <attribute name="PROD_ID" value="RES-07856" x="9.8425" y="10.16" size="1.778" layer="28" font="vector" ratio="15" rot="MR180" display="off"/>
@@
 <wire x1="46.99" y1="10.922" x2="47.244" y2="10.922" width="0.2032" layer="16"/>
 <wire x1="47.244" y1="10.922" x2="47.752" y2="10.414" width="0.2032" layer="16"/>
+<via x="32.131" y="6.985" extent="1-16" drill="0.381"/>
 </signal>
 <signal name="I2C_SDA">
@@
 <wire x1="23.495" y1="14.2875" x2="24.4475" y2="14.2875" width="0.2032" layer="1"/>
 <wire x1="24.4475" y1="14.2875" x2="25.0825" y2="13.6525" width="0.2032" layer="1"/>
-<via x="34.29" y="5.08" extent="1-16" drill="0.508" diameter="1.016"/>
+<via x="34.29" y="7.62" extent="1-16" drill="0.508" diameter="1.016"/>
 <wire x1="26.035" y1="12.065" x2="25.0825" y2="12.065" width="0.2032" layer="16"/>
 <wire x1="22.5425" y1="10.4775" x2="23.495" y2="10.4775" width="0.2032" layer="16"/>
-<wire x1="32.258" y1="12.192" x2="32.258" y2="6.604" width="0.2032" layer="16"/>
-<wire x1="32.258" y1="6.604" x2="33.782" y2="5.08" width="0.2032" layer="16"/>
-<wire x1="34.29" y1="5.08" x2="33.782" y2="5.08" width="0.2032" layer="16"/>
 <wire x1="22.255" y1="11.3633" x2="22.255" y2="10.765" width="0.2032" layer="16"/>
 <wire x1="22.255" y1="10.765" x2="22.5425" y2="10.4775" width="0.2032" layer="16"/>
@@
 <wire x1="29.337" y1="12.827" x2="31.623" y2="12.827" width="0.2032" layer="16"/>
 <wire x1="31.623" y1="12.827" x2="32.258" y2="12.192" width="0.2032" layer="16"/>
+<wire x1="32.258" y1="12.192" x2="32.258" y2="8.382" width="0.2032" layer="16"/>
+<wire x1="32.258" y1="8.382" x2="33.02" y2="7.62" width="0.2032" layer="16"/>
+<wire x1="33.02" y1="7.62" x2="34.29" y2="7.62" width="0.2032" layer="16"/>
 </signal>
 <signal name="ICSPCLK/DATA_RDY">
@@
 <contactref element="JP3" pad="1"/>
 <contactref element="TP4" pad="P$1"/>
-<via x="34.29" y="7.62" extent="1-16" drill="0.508" diameter="1.016"/>
+<via x="34.29" y="5.08" extent="1-16" drill="0.508" diameter="1.016"/>
 <wire x1="21.59" y1="13.208" x2="20.828" y2="12.446" width="0.2032" layer="1"/>
 <wire x1="23.622" y1="13.208" x2="21.59" y2="13.208" width="0.2032" layer="1"/>
@@
 <via x="20.828" y="12.446" extent="1-16" drill="0.381"/>
 <via x="23.622" y="13.208" extent="1-16" drill="0.381"/>
-<wire x1="33.274" y1="14.224" x2="33.274" y2="8.636" width="0.2032" layer="16"/>
-<wire x1="33.274" y1="8.636" x2="34.29" y2="7.62" width="0.2032" layer="16"/>
-<wire x1="34.29" y1="7.62" x2="35.052" y2="7.62" width="0.2032" layer="1"/>
-<wire x1="35.052" y1="7.62" x2="35.814" y2="6.858" width="0.2032" layer="1"/>
-<wire x1="35.814" y1="6.858" x2="35.814" y2="3.429" width="0.2032" layer="1"/>
-<wire x1="35.814" y1="3.429" x2="33.655" y2="1.27" width="0.2032" layer="1"/>
 <wire x1="21.605" y1="11.3633" x2="21.605" y2="12.304" width="0.2032" layer="16"/>
 <wire x1="21.605" y1="12.304" x2="21.463" y2="12.446" width="0.2032" layer="16"/>
 <wire x1="21.463" y1="12.446" x2="20.828" y2="12.446" width="0.2032" layer="16"/>
+<wire x1="33.655" y1="1.27" x2="33.655" y2="4.445" width="0.2032" layer="1"/>
+<wire x1="33.655" y1="4.445" x2="34.29" y2="5.08" width="0.2032" layer="1"/>
+<via x="34.417" y="8.763" extent="1-16" drill="0.381"/>
+<wire x1="33.274" y1="14.224" x2="33.274" y2="9.271" width="0.2032" layer="16"/>
+<wire x1="33.274" y1="9.271" x2="33.782" y2="8.763" width="0.2032" layer="16"/>
+<wire x1="33.782" y1="8.763" x2="34.417" y2="8.763" width="0.2032" layer="16"/>
+<wire x1="34.417" y1="8.763" x2="35.56" y2="7.62" width="0.2032" layer="1"/>
+<wire x1="35.56" y1="7.62" x2="35.56" y2="6.35" width="0.2032" layer="1"/>
+<wire x1="35.56" y1="6.35" x2="34.29" y2="5.08" width="0.2032" layer="1"/>
 </signal>
 <signal name="MCLR">
@@
 <wire x1="34.29" y1="14.224" x2="35.941" y2="12.573" width="0.2032" layer="16"/>
 <wire x1="35.941" y1="12.573" x2="35.941" y2="8.001" width="0.2032" layer="16"/>
-<wire x1="35.941" y1="8.001" x2="34.29" y2="6.35" width="0.2032" layer="16"/>
 <wire x1="34.29" y1="6.35" x2="33.528" y2="6.35" width="0.2032" layer="1"/>
 <wire x1="33.528" y1="6.35" x2="32.766" y2="5.588" width="0.2032" layer="1"/>
@@
 <wire x1="22.86" y1="2.667" x2="32.639" y2="2.667" width="0.2032" layer="16"/>
 <wire x1="32.639" y1="2.667" x2="32.766" y2="2.54" width="0.2032" layer="16"/>
+<wire x1="35.941" y1="8.001" x2="34.29" y2="6.35" width="0.2032" layer="16"/>
 </signal>
 <signal name="N$1">

Commit message: Updated Brd File
Routing:
- net GND: track 131.2 -> 130.9 mm, vias 19 -> 16
Changed lines of the file:
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@@
 <setting verticaltext="up"/>
 </settings>
-<grid distance="0.05" unitdist="inch" unit="inch" style="dots" multiple="1" display="yes" altdistance="0.005" altunitdist="inch" altunit="inch"/>
+<grid distance="0.025" unitdist="inch" unit="inch" style="dots" multiple="1" display="yes" altdistance="0.005" altunitdist="inch" altunit="inch"/>
 <layers>
 <layer number="1" name="Top" color="4" fill="1" visible="yes" active="yes"/>
-<layer number="2" name="Route2" color="1" fill="3" visible="yes" active="yes"/>
-<layer number="15" name="Route15" color="4" fill="6" visible="yes" active="yes"/>
+<layer number="2" name="Route2" color="1" fill="3" visible="no" active="yes"/>
+<layer number="15" name="Route15" color="4" fill="6" visible="no" active="yes"/>
 <layer number="16" name="Bottom" color="1" fill="1" visible="yes" active="yes"/>
 <layer number="17" name="Pads" color="2" fill="1" visible="yes" active="yes"/>
@@
 <layer number="23" name="tOrigins" color="15" fill="1" visible="yes" active="yes"/>
 <layer number="24" name="bOrigins" color="15" fill="1" visible="yes" active="yes"/>
-<layer number="25" name="tNames" color="7" fill="1" visible="yes" active="yes"/>
-<layer number="26" name="bNames" color="7" fill="1" visible="yes" active="yes"/>
-<layer number="27" name="tValues" color="7" fill="1" visible="yes" active="yes"/>
-<layer number="28" name="bValues" color="7" fill="1" visible="yes" active="yes"/>
-<layer number="29" name="tStop" color="7" fill="3" visible="yes" active="yes"/>
-<layer number="30" name="bStop" color="7" fill="6" visible="yes" active="yes"/>
-<layer number="31" name="tCream" color="7" fill="4" visible="yes" active="yes"/>
-<layer number="32" name="bCream" color="7" fill="5" visible="yes" active="yes"/>
-<layer number="39" name="tKeepout" color="4" fill="11" visible="yes" active="yes"/>
-<layer number="40" name="bKeepout" color="1" fill="11" visible="yes" active="yes"/>
-<layer number="41" name="tRestrict" color="4" fill="10" visible="yes" active="yes"/>
-<layer number="42" name="bRestrict" color="1" fill="10" visible="yes" active="yes"/>
-<layer number="43" name="vRestrict" color="2" fill="10" visible="yes" active="yes"/>
-<layer number="44" name="Drills" color="7" fill="1" visible="yes" active="yes"/>
+<layer number="25" name="tNames" color="7" fill="1" visible="no" active="yes"/>
+<layer number="26" name="bNames" color="7" fill="1" visible="no" active="yes"/>
+<layer number="27" name="tValues" color="7" fill="1" visible="no" active="yes"/>
+<layer number="28" name="bValues" color="7" fill="1" visible="no" active="yes"/>
+<layer number="29" name="tStop" color="7" fill="3" visible="no" active="yes"/>
+<layer number="30" name="bStop" color="7" fill="6" visible="no" active="yes"/>
+<layer number="31" name="tCream" color="7" fill="4" visible="no" active="yes"/>
+<layer number="32" name="bCream" color="7" fill="5" visible="no" active="yes"/>
+<layer number="39" name="tKeepout" color="4" fill="11" visible="no" active="yes"/>
+<layer number="40" name="bKeepout" color="1" fill="11" visible="no" active="yes"/>
+<layer number="41" name="tRestrict" color="4" fill="10" visible="no" active="yes"/>
+<layer number="42" name="bRestrict" color="1" fill="10" visible="no" active="yes"/>
+<layer number="43" name="vRestrict" color="2" fill="10" visible="no" active="yes"/>
+<layer number="44" name="Drills" color="7" fill="1" visible="no" active="yes"/>
 <layer number="45" name="Holes" color="7" fill="1" visible="yes" active="yes"/>
-<layer number="46" name="Milling" color="3" fill="1" visible="yes" active="yes"/>
-<layer number="47" name="Measures" color="7" fill="1" visible="yes" active="yes"/>
+<layer number="46" name="Milling" color="3" fill="1" visible="no" active="yes"/>
+<layer number="47" name="Measures" color="7" fill="1" visible="no" active="yes"/>
 <layer number="51" name="tDocu" color="6" fill="1" visible="yes" active="yes"/>
-<layer number="52" name="bDocu" color="7" fill="1" visible="yes" active="yes"/>
+<layer number="52" name="bDocu" color="7" fill="1" visible="no" active="yes"/>
 <layer number="3" name="Route3" color="4" fill="3" visible="no" active="no"/>
 <layer number="4" name="Route4" color="1" fill="4" visible="no" active="no"/>
@@
 <wire x1="22.905" y1="12.81375" x2="22.70125" y2="13.0175" width="0.2032" layer="16"/>
 <wire x1="22.70125" y1="13.0175" x2="21.2725" y2="13.0175" width="0.2032" layer="16"/>
-<via x="48.387" y="15.748" extent="1-16" drill="0.381"/>
 <wire x1="17.78" y1="14.9225" x2="18.796" y2="14.9225" width="0.2032" layer="16"/>
 <wire x1="18.796" y1="14.9225" x2="19.6215" y2="14.9225" width="0.2032" layer="16"/>
@@
 <wire x1="31.496" y1="10.16" x2="29.718" y2="8.382" width="0.2032" layer="1"/>
 <wire x1="30.099" y1="7.774" x2="30.075" y2="7.75" width="0.2032" layer="1"/>
-<wire x1="51.689" y1="3.429" x2="51.689" y2="8.382" width="0.2032" layer="1"/>
-<wire x1="47.625" y1="3.429" x2="51.689" y2="3.429" width="0.2032" layer="16"/>
-<wire x1="47.625" y1="9.525" x2="47.625" y2="3.429" width="0.2032" layer="1"/>
-<wire x1="47.752" y1="9.652" x2="47.625" y2="9.525" width="0.2032" layer="16"/>
-<wire x1="47.752" y1="10.414" x2="47.752" y2="9.652" width="0.2032" layer="16"/>
-<via x="51.689" y="8.382" extent="1-16" drill="0.381"/>
-<via x="51.689" y="3.429" extent="1-16" drill="0.381"/>
-<via x="47.625" y="3.429" extent="1-16" drill="0.381"/>
-<via x="47.625" y="9.525" extent="1-16" drill="0.381"/>
-<wire x1="47.625" y1="9.525" x2="47.625" y2="14.986" width="0.2032" layer="1"/>
-<wire x1="47.625" y1="14.986" x2="48.387" y2="15.748" width="0.2032" layer="1"/>
-<wire x1="47.752" y1="8.255" x2="47.752" y2="9.525" width="0.2032" layer="16"/>
-<wire x1="46.99" y1="7.493" x2="47.752" y2="8.255" width="0.2032" layer="16"/>
-<wire x1="36.703" y1="7.493" x2="46.99" y2="7.493" width="0.2032" layer="16"/>
-<wire x1="47.752" y1="9.525" x2="47.625" y2="9.525" width="0.2032" layer="16"/>
-<via x="36.703" y="7.493" extent="1-16" drill="0.381"/>
-<wire x1="34.29" y1="10.16" x2="35.814" y2="10.16" width="0.2032" layer="1"/>
-<wire x1="35.814" y1="10.16" x2="36.703" y2="9.271" width="0.2032" layer="1"/>
-<wire x1="36.703" y1="9.271" x2="36.703" y2="7.493" width="0.2032" layer="1"/>
 <via x="31.877" y="15.24" extent="1-16" drill="0.381"/>
 <wire x1="20.955" y1="14.39" x2="20.955" y2="15.113" width="0.2032" layer="16"/>
@@
 <wire x1="26.543" y1="15.367" x2="26.67" y2="15.24" width="0.2032" layer="16"/>
 <via x="32.512" y="13.462" extent="1-16" drill="0.381"/>
-<wire x1="51.689" y1="8.382" x2="50.7755" y2="8.382" width="0.2032" layer="16"/>
-<wire x1="50.7755" y1="8.382" x2="50.4825" y2="8.675" width="0.2032" layer="16"/>
 <wire x1="7.62" y1="8.636" x2="9.4615" y2="8.636" width="0.2032" layer="16"/>
 <wire x1="9.4615" y1="8.636" x2="9.525" y2="8.5725" width="0.2032" layer="16"/>
@@
 <wire x1="31.877" y1="14.097" x2="32.512" y2="13.462" width="0.2032" layer="1"/>
 <wire x1="32.512" y1="13.462" x2="32.512" y2="10.16" width="0.2032" layer="1"/>
-<wire x1="46.7425" y1="11.1125" x2="46.7995" y2="11.1125" width="0.2032" layer="16"/>
-<wire x1="46.7995" y1="11.1125" x2="46.99" y2="10.922" width="0.2032" layer="16"/>
-<wire x1="46.99" y1="10.922" x2="47.244" y2="10.922" width="0.2032" layer="16"/>
-<wire x1="47.244" y1="10.922" x2="47.752" y2="10.414" width="0.2032" layer="16"/>
 <via x="32.131" y="6.985" extent="1-16" drill="0.381"/>
+<via x="52.07" y="8.89" extent="1-16" drill="0.381"/>
+<wire x1="46.7425" y1="11.1125" x2="46.9265" y2="11.1125" width="0.2032" layer="16"/>
+<wire x1="46.9265" y1="11.1125" x2="47.625" y2="10.414" width="0.2032" layer="16"/>
+<wire x1="47.625" y1="10.414" x2="47.625" y2="8.89" width="0.2032" layer="16"/>
+<wire x1="47.625" y1="8.89" x2="45.72" y2="6.985" width="0.2032" layer="16"/>
+<wire x1="30.099" y1="6.223" x2="31.369" y2="6.223" width="0.2032" layer="1"/>
+<wire x1="31.369" y1="6.223" x2="32.131" y2="6.985" width="0.2032" layer="1"/>
+<wire x1="34.29" y1="10.16" x2="36.83" y2="10.16" width="0.2032" layer="1"/>
+<wire x1="36.83" y1="10.16" x2="40.64" y2="6.35" width="0.2032" layer="1"/>
+<via x="40.64" y="6.35" extent="1-16" drill="0.381"/>
+<wire x1="45.72" y1="6.985" x2="41.275" y2="6.985" width="0.2032" layer="16"/>
+<wire x1="41.275" y1="6.985" x2="40.64" y2="6.35" width="0.2032" layer="16"/>
+<wire x1="50.4825" y1="8.675" x2="51.855" y2="8.675" width="0.2032" layer="16"/>
+<wire x1="51.855" y1="8.675" x2="52.07" y2="8.89" width="0.2032" layer="16"/>
+<wire x1="52.07" y1="8.89" x2="52.07" y2="4.445" width="0.2032" layer="1"/>
+<wire x1="52.07" y1="4.445" x2="49.53" y2="1.905" width="0.2032" layer="1"/>
+<wire x1="49.53" y1="1.905" x2="43.815" y2="1.905" width="0.2032" layer="1"/>
+<wire x1="43.815" y1="1.905" x2="40.64" y2="5.08" width="0.2032" layer="1"/>
+<wire x1="40.64" y1="5.08" x2="40.64" y2="6.35" width="0.2032" layer="1"/>
+<via x="48.26" y="15.875" extent="1-16" drill="0.381"/>
 </signal>
 <signal name="I2C_SDA">
