File: Hardware/ZX_Gesture_Sensor_SMD_v02.brd (EAGLE design)
At the start: 57.2 x 19.1 mm, 51 parts, among them Q1 MMBT2222A, Q2 MOSFET-NCHANNEL2N7002PW, U1 PIC16F1823-14PINTSSOP, U2 MCP6021T-E/OT, U3 DMC2700UDM, U4 DMC2700UDM, U6 TSOP57238TT1

Commit message: Updated brd file
Parts:
- moved U$5 17.8 mm to (31.1, 7.20)
- moved U$6 17.8 mm to (14.4, 6.22)
- moved U$1 9.50 mm to (43.1, 15.9), turned to 270 degrees
- moved LOGO2 1.63 mm to (9.33, 2.20)
Routing:
- net N$2: track 21.7 -> 11.2 mm
- net GND: track 130.9 -> 128.8 mm
Other:
- board text added: "All Units Inches"

Commit message: Updated brd file
Routing:
- net VCC: track 104.5 -> 105.6 mm
Changed lines of the file:
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@@
 <setting verticaltext="up"/>
 </settings>
-<grid distance="0.025" unitdist="inch" unit="inch" style="dots" multiple="1" display="yes" altdistance="0.005" altunitdist="inch" altunit="inch"/>
+<grid distance="0.01" unitdist="inch" unit="inch" style="dots" multiple="1" display="yes" altdistance="0.005" altunitdist="inch" altunit="inch"/>
 <layers>
 <layer number="1" name="Top" color="4" fill="1" visible="yes" active="yes"/>
-<layer number="2" name="Route2" color="1" fill="3" visible="yes" active="yes"/>
-<layer number="15" name="Route15" color="4" fill="6" visible="yes" active="yes"/>
+<layer number="2" name="Route2" color="1" fill="3" visible="no" active="yes"/>
+<layer number="15" name="Route15" color="4" fill="6" visible="no" active="yes"/>
 <layer number="16" name="Bottom" color="1" fill="1" visible="yes" active="yes"/>
 <layer number="17" name="Pads" color="2" fill="1" visible="yes" active="yes"/>
@@
 <layer number="23" name="tOrigins" color="15" fill="1" visible="yes" active="yes"/>
 <layer number="24" name="bOrigins" color="15" fill="1" visible="yes" active="yes"/>
-<layer number="25" name="tNames" color="7" fill="1" visible="yes" active="yes"/>
-<layer number="26" name="bNames" color="7" fill="1" visible="yes" active="yes"/>
-<layer number="27" name="tValues" color="7" fill="1" visible="yes" active="yes"/>
-<layer number="28" name="bValues" color="7" fill="1" visible="yes" active="yes"/>
-<layer number="29" name="tStop" color="7" fill="3" visible="yes" active="yes"/>
-<layer number="30" name="bStop" color="7" fill="6" visible="yes" active="yes"/>
-<layer number="31" name="tCream" color="7" fill="4" visible="yes" active="yes"/>
-<layer number="32" name="bCream" color="7" fill="5" visible="yes" active="yes"/>
-<layer number="39" name="tKeepout" color="4" fill="11" visible="yes" active="yes"/>
-<layer number="40" name="bKeepout" color="1" fill="11" visible="yes" active="yes"/>
-<layer number="41" name="tRestrict" color="4" fill="10" visible="yes" active="yes"/>
-<layer number="42" name="bRestrict" color="1" fill="10" visible="yes" active="yes"/>
-<layer number="43" name="vRestrict" color="2" fill="10" visible="yes" active="yes"/>
-<layer number="44" name="Drills" color="7" fill="1" visible="yes" active="yes"/>
+<layer number="25" name="tNames" color="7" fill="1" visible="no" active="yes"/>
+<layer number="26" name="bNames" color="7" fill="1" visible="no" active="yes"/>
+<layer number="27" name="tValues" color="7" fill="1" visible="no" active="yes"/>
+<layer number="28" name="bValues" color="7" fill="1" visible="no" active="yes"/>
+<layer number="29" name="tStop" color="7" fill="3" visible="no" active="yes"/>
+<layer number="30" name="bStop" color="7" fill="6" visible="no" active="yes"/>
+<layer number="31" name="tCream" color="7" fill="4" visible="no" active="yes"/>
+<layer number="32" name="bCream" color="7" fill="5" visible="no" active="yes"/>
+<layer number="39" name="tKeepout" color="4" fill="11" visible="no" active="yes"/>
+<layer number="40" name="bKeepout" color="1" fill="11" visible="no" active="yes"/>
+<layer number="41" name="tRestrict" color="4" fill="10" visible="no" active="yes"/>
+<layer number="42" name="bRestrict" color="1" fill="10" visible="no" active="yes"/>
+<layer number="43" name="vRestrict" color="2" fill="10" visible="no" active="yes"/>
+<layer number="44" name="Drills" color="7" fill="1" visible="no" active="yes"/>
 <layer number="45" name="Holes" color="7" fill="1" visible="yes" active="yes"/>
-<layer number="46" name="Milling" color="3" fill="1" visible="yes" active="yes"/>
-<layer number="47" name="Measures" color="7" fill="1" visible="yes" active="yes"/>
+<layer number="46" name="Milling" color="3" fill="1" visible="no" active="yes"/>
+<layer number="47" name="Measures" color="7" fill="1" visible="no" active="yes"/>
 <layer number="51" name="tDocu" color="6" fill="1" visible="yes" active="yes"/>
-<layer number="52" name="bDocu" color="7" fill="1" visible="yes" active="yes"/>
+<layer number="52" name="bDocu" color="7" fill="1" visible="no" active="yes"/>
 <layer number="3" name="Route3" color="4" fill="3" visible="no" active="no"/>
 <layer number="4" name="Route4" color="1" fill="4" visible="no" active="no"/>
@@
 <wire x1="12.065" y1="10.795" x2="11.7475" y2="11.1125" width="0.2032" layer="16"/>
 <wire x1="25.82" y1="11.1125" x2="25.7175" y2="11.01" width="0.2032" layer="1"/>
-<wire x1="25.7175" y1="11.01" x2="26.5675" y2="11.01" width="0.2032" layer="1"/>
-<wire x1="27.075" y1="11.3" x2="26.8575" y2="11.3" width="0.2032" layer="1"/>
-<wire x1="26.8575" y1="11.3" x2="26.5675" y2="11.01" width="0.2032" layer="1"/>
 <wire x1="50.165" y1="11.43" x2="50.165" y2="11.049" width="0.2032" layer="16"/>
 <wire x1="50.165" y1="11.049" x2="50.165" y2="10.6925" width="0.2032" layer="16"/>
 <wire x1="50.165" y1="10.6925" x2="50.4825" y2="10.375" width="0.2032" layer="16"/>
 <wire x1="50.1015" y1="11.1125" x2="50.165" y2="11.049" width="0.2032" layer="16"/>
-<wire x1="27.075" y1="11.3" x2="27.075" y2="15.089" width="0.2032" layer="1"/>
+<wire x1="27.075" y1="11.3" x2="27.075" y2="12.446" width="0.2032" layer="1"/>
+<wire x1="27.075" y1="12.446" x2="27.075" y2="15.089" width="0.2032" layer="1"/>
 <wire x1="27.075" y1="15.089" x2="26.67" y2="15.494" width="0.2032" layer="1"/>
 <wire x1="26.67" y1="15.494" x2="25.4" y2="15.494" width="0.2032" layer="1"/>
@@
 <wire x1="15.0876" y1="12.3952" x2="16.1798" y2="12.3952" width="0.2032" layer="16"/>
 <wire x1="16.1798" y1="12.3952" x2="16.1925" y2="12.3825" width="0.2032" layer="16"/>
+<wire x1="25.7175" y1="11.01" x2="25.7175" y2="12.0015" width="0.2032" layer="1"/>
+<wire x1="25.7175" y1="12.0015" x2="26.162" y2="12.446" width="0.2032" layer="1"/>
+<wire x1="26.162" y1="12.446" x2="27.075" y2="12.446" width="0.2032" layer="1"/>
 </signal>
 <signal name="GND">
