File: Hardware/ZX_Gesture_Sensor_SMD_v03.sch (EAGLE design)
At the start: 50 parts, among them Q1 MMBT2222A, Q2 MOSFET-NCHANNEL2N7002PW, U1 PIC16F1823-14PINTSSOP, U2 MCP6021T-E/OT, U3 DMC2700UDM, U4 DMC2700UDM, U6 TSOP57238TT1

Commit message: Updated Brd and Sch Files per QC review
Parts:
- R3: device SparkFun-Resistors:10OHM-1/10W-1%(0603)SMD -> SparkFun-Resistors:10OHM-1/10W-5%0603SMD; TOL 1% -> (none)
- renumbered JP3 to JP2, U6 to U5
Connections:
- net GND: now also TP3.1; no longer TP2.1
- net ICSPCLK/DATA_RDY: now also TP5.1; no longer TP4.1
- net ICSPDAT/DACOUT: now also TP4.1; no longer TP5.1
- net MCLR: now also TP1.1; no longer TP3.1
- net VCC: now also TP2.1; no longer TP1.1
Other:
- moved on the sheet: TP1, TP2, TP3, TP4, TP5
